Commit message: added launch file to shorten commands

File: install/ana/share/ana/description/robot_core.xacro (robot description, xacro)
@@ -21,5 +21,5 @@
         <parent link="base_link"/>
         <child link="chassis"/>
-        <origin xyz="-0.1 0 0"/> <!-- behind base link -->
+        <origin xyz="-0.001 0 0"/>
     </joint>
     <link name="chassis">
@@ -45,5 +45,5 @@
         <parent link="base_link"/>
         <child link="front_left_wheel"/>
-        <origin xyz="0.005 0.098 0" rpy="-1.5708 0 0"/>
+        <origin xyz="0.104 0.098 0" rpy="-1.5708 0 0"/>
         <axis xyz="0 0 1"/>
     </joint>
@@ -68,5 +68,5 @@
         <parent link="base_link"/>
         <child link="front_right_wheel"/>
-        <origin xyz="-0.005 -0.101 0" rpy="1.5708 0 0"/>
+        <origin xyz="0.094 -0.101 0" rpy="1.5708 0 0"/>
         <axis xyz="0 0 -1"/>
     </joint>
@@ -91,5 +91,5 @@
         <parent link="base_link"/>
         <child link="back_left_wheel"/>
-        <origin xyz="-0.203 0.098 0" rpy="-1.5708 0 0"/>
+        <origin xyz="-0.104 0.098 0" rpy="-1.5708 0 0"/>
         <axis xyz="0 0 1"/>
     </joint>
@@ -114,5 +114,5 @@
         <parent link="base_link"/>
         <child link="back_right_wheel"/>
-        <origin xyz="-0.203 -0.101 0" rpy="1.5708 0 0"/>
+        <origin xyz="-0.104 -0.101 0" rpy="1.5708 0 0"/>
         <axis xyz="0 0 -1"/>
     </joint>
