Commit message: Simulation Xacros, Differential Drive

File: install/ana/share/ana/description/robot.urdf.xacro (robot description, xacro)
@@ -3,3 +3,4 @@
     <!-- Example Link -->
     <xacro:include filename="robot_core.xacro" />
+    <xacro:include filename="gazebo_diff_control.xacro"/>
 </robot>

File: install/ana/share/ana/description/robot_core.xacro (robot description, xacro)
@@ -29,5 +29,5 @@
                 <mesh filename="file:///home/aidanr/R2G_robot/src/ana/meshes/ana_chassis.stl" scale="0.001 0.001 0.001"/>
             </geometry>
-            <material name="white"/>
+            <material name="blue"/>
         </visual>
         <collision>
@@ -41,4 +41,7 @@
         </xacro:inertial_box>
     </link>
+    <gazebo reference="chassis">
+        <material>Gazebo/Blue</material>
+    </gazebo>
     <!-- FRONT LEFT WHEEL LINK -->
     <joint name="front_left_wheel_joint" type="continuous">
@@ -64,4 +67,7 @@
         </xacro:inertial_cylinder>
     </link>
+    <gazebo reference="front_left_wheel">
+        <material>Gazebo/Black</material>
+    </gazebo>
     <!-- FRONT RIGHT WHEEL LINK -->
     <joint name="front_right_wheel_joint" type="continuous">
@@ -87,4 +93,7 @@
         </xacro:inertial_cylinder>
     </link>
+    <gazebo reference="front_right_wheel">
+        <material>Gazebo/Black</material>
+    </gazebo>
     <!-- BACK LEFT WHEEL LINK -->
     <joint name="back_left_wheel_joint" type="continuous">
@@ -110,4 +119,7 @@
         </xacro:inertial_cylinder>
     </link>
+    <gazebo reference="back_left_wheel">
+        <material>Gazebo/Black</material>
+    </gazebo>
     <!-- BACK RIGHT WHEEL LINK -->
     <joint name="back_right_wheel_joint" type="continuous">
@@ -133,3 +145,6 @@
         </xacro:inertial_cylinder>
     </link>
+    <gazebo reference="back_right_wheel">
+        <material>Gazebo/Black</material>
+    </gazebo>
 </robot>

File: src/ana/description/robot.urdf.xacro (robot description, xacro)
@@ -3,3 +3,4 @@
     <!-- Example Link -->
     <xacro:include filename="robot_core.xacro" />
+    <xacro:include filename="gazebo_diff_control.xacro"/>
 </robot>
