Commit message: rtab-map filtered and published to rviz2

File: install/ana/share/ana/description/camera.xacro (robot description, xacro)
@@ -12,5 +12,7 @@
                 <mesh filename="file:///home/aidan/ana_bot/src/ana/meshes/d435i.stl"/>
             </geometry>
-            <material name="red"/>
+            <material name="grey">
+                <color rgba="0.5 0.5 0.5 1.0"/> <!-- Define grey color in RGBA format -->
+            </material>
         </visual>
     </link>

File: install/ana/share/ana/description/depth_camera.xacro (robot description, xacro)
@@ -12,5 +12,7 @@
                 <mesh filename="file:///home/aidan/ana_bot/src/ana/meshes/d435i.stl"/>
             </geometry>
-            <material name="red"/>
+            <material name="grey">
+                <color rgba="0.5 0.5 0.5 1.0"/> <!-- Define grey color in RGBA format -->
+            </material>
         </visual>
     </link>
