Commit message: SLAM, Costmap generation

File: src/ana/description/depth_camera.xacro (robot description, xacro)
@@ -34,6 +34,6 @@
                 <image>
                     <format>B8G8R8</format>
-                    <width>640</width>
-                    <height>480</height> <!-- Lower resolution for faster processing -->
+                    <width>1280</width>
+                    <height>720</height> <!-- Lower resolution for faster processing -->
                 </image>
                 <!-- filter for min max ranges -->

File: src/ana/description/robot_core.xacro (robot description, xacro)
@@ -17,4 +17,5 @@
     <!-- CHASSIS LINK -->
     <link name="base_link">
+        <origin xyz="0 0 0"/>
     </link>
     <joint name="chassis_joint" type="fixed">
