Commit message: lowered drift between gazebo and rviz car

File: src/ana/description/robot_core.xacro (robot description, xacro)
@@ -60,5 +60,5 @@
         <collision>
             <geometry>
-                <cylinder radius="0.0325" length="0.027" />
+                <sphere radius="0.0325"/> <!-- reduces chances of gazebo/rviz car location drift (friction) -->
             </geometry>
         </collision>
@@ -86,5 +86,5 @@
         <collision>
             <geometry>
-                <cylinder radius="0.0325" length="0.027" />
+                <sphere radius="0.0325"/>
             </geometry>
         </collision>
@@ -112,5 +112,5 @@
         <collision>
             <geometry>
-                <cylinder radius="0.0325" length="0.027" />
+                <sphere radius="0.0325"/>
             </geometry>
         </collision>
@@ -121,6 +121,6 @@
     <gazebo reference="back_left_wheel">
         <material>Gazebo/Black</material>
-        <mu1 value="0.001"/>
-        <mu2 value="0.001"/>
+        <!-- <mu1 value="0.001"/>
+        <mu2 value="0.001"/> -->
     </gazebo>
     <!-- BACK RIGHT WHEEL LINK -->
@@ -140,5 +140,5 @@
         <collision>
             <geometry>
-                <cylinder radius="0.0325" length="0.027" />
+                <sphere radius="0.0325"/>
             </geometry>
         </collision>
@@ -149,6 +149,6 @@
     <gazebo reference="back_right_wheel">
         <material>Gazebo/Black</material>
-        <mu1 value="0.001"/>
-        <mu2 value="0.001"/>
+        <!-- <mu1 value="0.001"/>
+        <mu2 value="0.001"/> -->
     </gazebo>
 </robot>

File: src/ana/description/ros2_diff_control.xacro (robot description, xacro)
@@ -21,4 +21,20 @@
             <state_interface name="position"/>
         </joint>
+        <joint name="back_left_wheel_joint">
+        <command_interface name="velocity">
+            <param name="min">-10</param>
+            <param name="max">10</param>
+        </command_interface>
+        <state_interface name="velocity"/>
+        <state_interface name="position"/>
+        </joint>
+        <joint name="back_right_wheel_joint">
+            <command_interface name="velocity">
+                <param name="min">-10</param>
+                <param name="max">10</param>
+            </command_interface>
+            <state_interface name="velocity"/>
+            <state_interface name="position"/>
+        </joint>
     </ros2_control>
     <gazebo>

Commit message: added skid steer for four wheels, RViz2 movement is smooth and Gazebo is not (TODO - fix gazebo)

File: src/ana/description/robot_core.xacro (robot description, xacro)
@@ -37,5 +37,5 @@
             </geometry>
         </collision>
-        <xacro:inertial_box mass="0.5" x="0.3" y="0.3" z="0.15"> <!-- kiligrams -->
+        <xacro:inertial_box mass="0.5" x="0.235" y="0.17" z="0.10"> <!-- kiligrams -->
             <origin xyz="0.1175 0.0835 0.0295" rpy="0 0 0"/>
         </xacro:inertial_box>
@@ -60,5 +60,5 @@
         <collision>
             <geometry>
-                <sphere radius="0.0325"/> <!-- reduces chances of gazebo/rviz car location drift (friction) -->
+                <cylinder radius="0.0325" length="0.027" />
             </geometry>
         </collision>
@@ -74,5 +74,5 @@
         <parent link="base_link"/>
         <child link="front_right_wheel"/>
-        <origin xyz="0.094 -0.1005 0" rpy="1.5708 0 0"/>
+        <origin xyz="0.104 -0.1005 0" rpy="1.5708 0 0"/>
         <axis xyz="0 0 -1"/>
     </joint>
@@ -86,5 +86,5 @@
         <collision>
             <geometry>
-                <sphere radius="0.0325"/>
+                <cylinder radius="0.0325" length="0.027" />
             </geometry>
         </collision>
@@ -112,5 +112,5 @@
         <collision>
             <geometry>
-                <sphere radius="0.0325"/>
+                <cylinder radius="0.0325" length="0.027" />
             </geometry>
         </collision>
@@ -140,5 +140,5 @@
         <collision>
             <geometry>
-                <sphere radius="0.0325"/>
+                <cylinder radius="0.0325" length="0.027" />
             </geometry>
         </collision>

File: src/ana/description/ros2_diff_control.xacro (robot description, xacro)
@@ -21,13 +21,13 @@
             <state_interface name="position"/>
         </joint>
-        <joint name="back_left_wheel_joint">
-        <command_interface name="velocity">
-            <param name="min">-10</param>
-            <param name="max">10</param>
-        </command_interface>
-        <state_interface name="velocity"/>
-        <state_interface name="position"/>
+        <joint name = "back_left_wheel_joint">
+            <command_interface name="velocity">
+                <param name="min">-10</param>
+                <param name="max">10</param>
+            </command_interface>
+            <state_interface name="velocity"/>
+            <state_interface name="position"/>
         </joint>
-        <joint name="back_right_wheel_joint">
+        <joint name = "back_right_wheel_joint">
             <command_interface name="velocity">
                 <param name="min">-10</param>

Commit message: goodbye

File: src/ana/description/robot_core.xacro (robot description, xacro)
@@ -37,5 +37,5 @@
             </geometry>
         </collision>
-        <xacro:inertial_box mass="0.5" x="0.235" y="0.17" z="0.10"> <!-- kiligrams -->
+        <xacro:inertial_box mass="0.5" x="0.235" y="0.17" z="0.0"> <!-- kiligrams -->
             <origin xyz="0.1175 0.0835 0.0295" rpy="0 0 0"/>
         </xacro:inertial_box>
@@ -60,5 +60,5 @@
         <collision>
             <geometry>
-                <cylinder radius="0.0325" length="0.027" />
+                <sphere radius="0.0325"/>
             </geometry>
         </collision>
@@ -86,5 +86,5 @@
         <collision>
             <geometry>
-                <cylinder radius="0.0325" length="0.027" />
+                <sphere radius="0.0325"/>
             </geometry>
         </collision>
@@ -112,5 +112,5 @@
         <collision>
             <geometry>
-                <cylinder radius="0.0325" length="0.027" />
+                <sphere radius="0.0325"/>
             </geometry>
         </collision>
@@ -140,5 +140,5 @@
         <collision>
             <geometry>
-                <cylinder radius="0.0325" length="0.027" />
+                <sphere radius="0.0325"/>
             </geometry>
         </collision>

Commit message: working nav2

File: src/ana/description/robot_core.xacro (robot description, xacro)
@@ -18,4 +18,11 @@
     <link name="base_link">
         <origin xyz="0 0 0"/>
+    </link>
+    <joint name="base_footprint_joint" type="fixed">
+        <parent link="base_link"/>
+        <child link="base_footprint"/>
+        <origin xyz="0 0 0" rpy="0 0 0"/>
+    </joint>
+    <link name="base_footprint">
     </link>
     <joint name="chassis_joint" type="fixed">
