Commit message: Working in real-world

File: src/ana/description/camera.xacro (robot description, xacro)
@@ -23,28 +23,3 @@
     </joint>
     <link name="camera_link_optical"></link>
-    <gazebo reference="camera_link">
-        <material>Gazebo/Grey</material>
-        <sensor name="camera" type="camera">
-            <pose> 0 0 0 0 0 0 </pose>
-            <visualize>true</visualize>
-            <update_rate>10</update_rate>
-            <camera>
-                <!-- specific to D435i | radians -->
-                <horizontal_fov>1.501</horizontal_fov>
-                <image>
-                    <format>R8G8B8</format>
-                    <width>1920</width>
-                    <height>1080</height>
-                </image>
-                <!-- filter for min max ranges -->
-                <clip>
-                    <near>0.05</near>
-                    <far>8.0</far>
-                </clip>
-            </camera>
-            <plugin name="camera_controller" filename="libgazebo_ros_camera.so">
-                <frame_name>camera_link_optical</frame_name>
-            </plugin>
-        </sensor>
-    </gazebo>
 </robot>

File: src/ana/description/depth_camera.xacro (robot description, xacro)
@@ -23,55 +23,3 @@
     </joint>
     <link name="camera_link_optical"></link>
-    <gazebo reference="camera_link">
-        <material>Gazebo/Grey</material>
-        <sensor name="camera" type="depth">
-            <pose> 0 0 0 0 0 0 </pose>
-            <visualize>true</visualize>
-            <update_rate>5</update_rate> <!-- d435i: 90fps -->
-            <camera>
-                <!-- specific to D435i | radians -->
-                <horizontal_fov>1.518436</horizontal_fov>
-                <image>
-                    <format>B8G8R8</format>
-                    <width>1280</width> <!-- d435i: 1280x720 -->
-                    <height>720</height>
-                </image>
-                <!-- filter for min max ranges -->
-                <clip>
-                    <near>0.28</near> <!-- d435i: ideal range .3m to 3m | min: 0.28m-->
-                    <far>6.0</far>
-                    <!-- 6 IS TYPICAL SWEET SPOT
-                        2 to 4 meters: 2-3% loss
-                        4 to 6 meters: 3-5% loss
-                        6 to 10 meters: 5-10% loss
-                        -->
-                </clip>
-            </camera>
-            <plugin name="camera_controller" filename="libgazebo_ros_camera.so">
-                <frame_name>camera_link_optical</frame_name>
-                <min_depth>0.1</min_depth> <!-- d435i: <2% accuracy at 2m-->
-                <max_depth>100</max_depth>
-            </plugin>
-        </sensor>
-        <sensor name="rgb_camera" type="camera">
-            <pose>0 0 0 0 0 0</pose>
-            <visualize>true</visualize>
-            <update_rate>30</update_rate> <!-- Frame rate for RGB camera -->
-            <camera>
-                <horizontal_fov>1.204277</horizontal_fov> <!-- FOV for RGB: 69° in radians -->
-                <image>
-                    <format>B8G8R8</format>
-                    <width>1920</width> <!-- Resolution for RGB: 1920x1080 -->
-                    <height>1080</height>
-                </image>
-                <clip>
-                    <near>0.3</near> <!-- Ideal range start for RGB -->
-                    <far>3.0</far> <!-- Ideal range end for RGB -->
-                </clip>
-            </camera>
-            <plugin name="rgb_camera_controller" filename="libgazebo_ros_camera.so">
-                <frame_name>camera_link_optical</frame_name>
-            </plugin>
-        </sensor>
-    </gazebo>
 </robot>

File: src/ana/description/gazebo_diff_control.xacro (robot description, xacro)
@@ -1,23 +1,4 @@
 <?xml version="1.0"?>
 <robot xmlns:xacro="http://www.ros.org/wiki/xacro"  name="robot">
-    <gazebo>
-        <plugin name="diff_drive" filename="libgazebo_ros_diff_drive.so">
-            <!-- Wheel Information-->
-            <left_joint>front_left_wheel_joint</left_joint>
-            <right_joint>front_right_wheel_joint</right_joint>
-            <!-- <left_joint>back_left_wheel_joint</left_joint> -->
-            <!-- <right_joint>back_right_wheel_joint</right_joint> -->
-            <wheel_separation>0.188</wheel_separation>
-            <wheel_diameter>0.065</wheel_diameter>
-            <!-- Limits -->
-            <max_wheel_torque>200</max_wheel_torque>
-            <max_wheel_acceleration>10.0</max_wheel_acceleration>
-            <!-- Outputs -->
-            <odometry_frame>odom</odometry_frame>
-            <robot_base_frame>base_link</robot_base_frame>
-            <publish_odom>true</publish_odom>
-            <publish_odom_tf>true</publish_odom_tf>
-            <publish_wheel_tf>true</publish_wheel_tf>
-        </plugin>
-    </gazebo>
+    <!-- This entire block is specific to Gazebo and not needed in real-world applications -->
 </robot>

File: src/ana/description/gazebo_four_diff_control.xacro (robot description, xacro)
@@ -1,28 +1,4 @@
 <?xml version="1.0"?>
 <robot xmlns:xacro="http://www.ros.org/wiki/xacro"  name="robot">
-    <gazebo>
-        <plugin name="skid_steer_drive" filename="libgazebo_ros_diff_drive.so">
-            <ros>
-                <namespace>/</namespace>
-                <remapping>cmd_vel:=cmd_vel</remapping>
-            </ros>
-            <update_rate>100.0</update_rate>
-            <num_wheel_pairs>2</num_wheel_pairs>
-            <left_joint>front_left_wheel_joint</left_joint>
-            <left_joint>back_left_wheel_joint</left_joint>
-            <right_joint>front_right_wheel_joint</right_joint>
-            <right_joint>back_right_wheel_joint</right_joint>
-            <wheel_separation>0.188</wheel_separation>
-            <wheel_separation>0.188</wheel_separation>
-            <wheel_diameter>0.065</wheel_diameter>
-            <wheel_diameter>0.065</wheel_diameter>
-            <max_wheel_torque>200.0</max_wheel_torque>
-            <max_wheel_acceleration>10.0</max_wheel_acceleration>
-            <odometry_frame>odom</odometry_frame>
-            <robot_base_frame>base_link</robot_base_frame>
-            <publish_odom>true</publish_odom>
-            <publish_odom_tf>true</publish_odom_tf>
-            <publish_wheel_tf>true</publish_wheel_tf>
-        </plugin>
-    </gazebo>
+    <!-- This entire block is specific to Gazebo and not needed in real-world applications -->
 </robot>

File: src/ana/description/livox_mid_360.xacro (robot description, xacro)
@@ -16,40 +16,3 @@
       </visual>
   </link>
-  <gazebo reference="livox_lidar">
-      <material>Gazebo/Blue</material>
-      <sensor name="livox_lidar_sensor" type="gpu_ray">
-          <pose>0 0 0 0 0 0</pose>
-          <!-- <visualize>false</visualize> visualize lasers -->
-          <update_rate>10</update_rate>
-          <ray>
-              <scan>
-                  <horizontal>
-                      <samples>3600</samples> <!-- Increased to simulate higher point density -->
-                      <resolution>1</resolution>
-                      <min_angle>-3.14159</min_angle> <!-- -180 degrees in radians -->
-                      <max_angle>3.14159</max_angle> <!-- 180 degrees in radians -->
-                  </horizontal>
-                  <vertical>
-                      <samples>59</samples> <!-- total degrees -->
-                      <resolution>1</resolution>
-                      <min_angle>-0.1222</min_angle> <!-- -7 degrees in radians -->
-                      <max_angle>0.9076</max_angle> <!-- 52 degrees in radians -->
-                  </vertical>
-              </scan>
-              <range>
-                  <min>0.17</min> <!-- depth camera is .1246 meters away -->
-                  <max>70.0</max> <!-- Maximum range at 80% reflectivity -->
-                  <resolution>0.01</resolution>
-              </range>
-          </ray>
-          <noise>
-              <mean>0.0</mean>
-              <stddev>0.02</stddev> <!-- Random error standard deviation -->
-          </noise>
-          <plugin name="livox_gazebo_plugin" filename="libgazebo_ros_ray_sensor.so">
-              <topicName>/livox/scan</topicName>
-              <frameName>livox_lidar</frameName>
-          </plugin>
-      </sensor>
-  </gazebo>
 </robot>

File: src/ana/description/robot.urdf.xacro (robot description, xacro)
@@ -4,5 +4,5 @@
     <xacro:include filename="robot_core.xacro" />
     <!-- <xacro:include filename="gazebo_diff_control.xacro"/> -->
-    <xacro:include filename="gazebo_four_diff_control.xacro"/>
+    <!-- <xacro:include filename="gazebo_four_diff_control.xacro"/> -->
     <!-- <xacro:include filename="ros2_diff_control.xacro"/> -->
     <!-- <xacro:include filename="camera.xacro"/> -->

File: src/ana/description/robot_core.xacro (robot description, xacro)
@@ -50,7 +50,4 @@
         </xacro:inertial_box>
     </link>
-    <gazebo reference="chassis">
-        <material>Gazebo/Blue</material>
-    </gazebo>
     <!-- FRONT LEFT WHEEL LINK -->
     <joint name="front_left_wheel_joint" type="continuous">
@@ -76,7 +73,4 @@
         </xacro:inertial_cylinder>
     </link>
-    <gazebo reference="front_left_wheel">
-        <material>Gazebo/Black</material>
-    </gazebo>
     <!-- FRONT RIGHT WHEEL LINK -->
     <joint name="front_right_wheel_joint" type="continuous">
@@ -102,7 +96,4 @@
         </xacro:inertial_cylinder>
     </link>
-    <gazebo reference="front_right_wheel">
-        <material>Gazebo/Black</material>
-    </gazebo>
     <!-- BACK LEFT WHEEL LINK -->
     <joint name="back_left_wheel_joint" type="continuous">
@@ -128,9 +119,4 @@
         </xacro:inertial_cylinder>
     </link>
-    <gazebo reference="back_left_wheel">
-        <material>Gazebo/Black</material>
-        <!-- <mu1 value="0.001"/> -->          <!--friction does not want to work -->
-        <!-- <mu2 value="0.001"/> -->
-    </gazebo>
     <!-- BACK RIGHT WHEEL LINK -->
     <joint name="back_right_wheel_joint" type="continuous">
@@ -156,8 +142,3 @@
         </xacro:inertial_cylinder>
     </link>
-    <gazebo reference="back_right_wheel">
-        <material>Gazebo/Black</material>
-        <!-- <mu1 value="0.001"/> -->           <!--friction does not want to work -->
-        <!-- <mu2 value="0.001"/> -->
-    </gazebo>
 </robot>

File: src/ana/description/ros2_diff_control.xacro (robot description, xacro)
@@ -1,5 +1,5 @@
 <?xml version="1.0"?>
 <robot xmlns:xacro="http://www.ros.org/wiki/xacro"  name="robot">
-    <ros2_control name="GazeboSystem" type="system">
+    <!-- <ros2_control name="GazeboSystem" type="system">
         <hardware>
             <plugin>gazebo_ros2_control/GazeboSystem</plugin>
@@ -42,4 +42,4 @@
             <parameters>$(find ana)/config/my_controllers.yaml</parameters>
         </plugin>
-    </gazebo>
+    </gazebo> -->
 </robot>
