Commit message: Physical Robot

File: src/ana/description/robot.urdf.xacro (robot description, xacro)
@@ -8,4 +8,5 @@
     <!-- <xacro:include filename="camera.xacro"/> -->
     <xacro:include filename="depth_camera.xacro"/>
-    <xacro:include filename="livox_mid_360.xacro"/>
+    <!-- <xacro:include filename="livox_mid_360.xacro"/> -->
+    <xacro:include filename="velodyne_vlp16.xacro"/>
 </robot>

File: src/ana/description/robot_core.xacro (robot description, xacro)
@@ -38,5 +38,5 @@
                 <mesh filename="file:///home/aidan/ana_bot/src/ana/meshes/ana_chassis.stl" scale="0.001 0.001 0.001"/>
             </geometry>
-            <material name="blue"/>
+            <material name="white"/>
         </visual>
         <collision>
